Commit message: scan

File: description/lidar.xacro (robot description, xacro)
@@ -23,5 +23,4 @@
     </link>
 <gazebo reference="laser_frame">
-<material>Gazebo/Red</material>
   <sensor name="laser" type="ray">
     <pose> 0 0 0 0 0 0 </pose>

Commit message: scan

File: description/lidar.xacro (robot description, xacro)
@@ -23,4 +23,5 @@
     </link>
 <gazebo reference="laser_frame">
+<material>Gazebo/Red</material>
   <sensor name="laser" type="ray">
     <pose> 0 0 0 0 0 0 </pose>
